File: emc_test.kicad_pcb (KiCad board)
At the start: 2 copper layers, 101 x 50 mm, 49 parts, among them J1 MSTBA_3C_5.08_Angled, J4 MSTBA_3C_5.08_Angled, X1 PE, X2 PE

Commit message: smulkus pataisymai
Parts:
- R14: value {R} -> 910R
Connections:
- C4 pad 1: Net-(C4-Pad1) -> /LOUT
- C5 pad 2: Net-(C5-Pad2) -> /NOUT
- J4 pad 1: Net-(C4-Pad1) -> /NOUT
- J4 pad 2: Net-(C5-Pad2) -> /LOUT
- L1 pad 2: Net-(C4-Pad1) -> /LOUT
- L2 pad 2: Net-(C5-Pad2) -> /NOUT
Routing:
- net Net-(C5-Pad2): track 10.6 -> 0.00 mm
- net /NOUT: track 0.00 -> 10.6 mm
- net Net-(C4-Pad1): track 10.5 -> 0.00 mm
- net /LOUT: track 0.00 -> 10.5 mm
- removed copper zone on F.Cu, net Net-(C4-Pad1)
- removed copper zone on F.Cu, net Net-(C5-Pad2)
Changed lines of the file:
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@@
   (general
     (links 96)
-    (no_connects 0)
-    (area 82.150001 68.3 208.557143 131.700001)
+    (no_connects 2)
+    (area 97.924999 73.924999 199.075001 124.075001)
     (thickness 1.6)
     (drawings 12)
@@
   (net 10 "Net-(D3-Pad1)")
   (net 11 "Net-(R1-Pad2)")
-  (net 12 "Net-(C4-Pad1)")
-  (net 13 "Net-(C5-Pad2)")
-  (net 14 /OUT)
+  (net 12 /OUT)
+  (net 13 /LOUT)
+  (net 14 /NOUT)
   (net_class Default "This is the default net class."
     (clearance 0.2)
@@
     (uvia_drill 0.1)
     (add_net /LINE)
+    (add_net /LOUT)
     (add_net /NEU)
+    (add_net /NOUT)
     (add_net /OUT)
     (add_net Earth)
     (add_net "Net-(C3-Pad1)")
     (add_net "Net-(C3-Pad2)")
-    (add_net "Net-(C4-Pad1)")
     (add_net "Net-(C4-Pad2)")
     (add_net "Net-(C5-Pad1)")
-    (add_net "Net-(C5-Pad2)")
     (add_net "Net-(C6-Pad2)")
     (add_net "Net-(D1-Pad1)")
@@
     )
     (pad 1 thru_hole circle (at 0 0 180) (size 2 2) (drill 1.00076) (layers *.Cu *.Mask)
-      (net 14 /OUT))
+      (net 12 /OUT))
   )
   (module Wire_Pads:SolderWirePad_single_1mmDrill (layer F.Cu)
@@
     )
     (pad 1 thru_hole circle (at 0 0 180) (size 2 2) (drill 1.00076) (layers *.Cu *.Mask)
-      (net 14 /OUT))
+      (net 12 /OUT))
   )
   (module Resistors_THT:R_Axial_DIN0207_L6.3mm_D2.5mm_P10.16mm_Horizontal (layer F.Cu)
@@
       (effects (font (size 1 1) (thickness 0.15)))
     )
-    (fp_text value {R} (at 5.08 2.31) (layer F.Fab)
+    (fp_text value 910R (at 5.08 2.31) (layer F.Fab)
       (effects (font (size 1 1) (thickness 0.15)))
     )
@@
       (net 2 Earth))
     (pad 2 thru_hole circle (at 10.16 0) (size 2 2) (drill 1) (layers *.Cu *.Mask)
-      (net 14 /OUT))
+      (net 12 /OUT))
     (model ${KISYS3DMOD}/Resistors_THT.3dshapes/R_Axial_DIN0207_L6.3mm_D2.5mm_P10.16mm_Horizontal.wrl
       (at (xyz 0 0 0))
@@
     )
     (pad 1 thru_hole rect (at 0 0 90) (size 2.4 4.8) (drill 1.4) (layers *.Cu *.Mask)
-      (net 12 "Net-(C4-Pad1)"))
+      (net 14 /NOUT))
     (pad 2 thru_hole oval (at 5.08 0 90) (size 2.4 4.8) (drill 1.4) (layers *.Cu *.Mask)
-      (net 13 "Net-(C5-Pad2)"))
+      (net 13 /LOUT))
     (pad 3 thru_hole oval (at 10.16 0 90) (size 2.4 4.8) (drill 1.4) (layers *.Cu *.Mask)
       (net 2 Earth))
@@
       (net 7 "Net-(C5-Pad1)"))
     (pad 2 thru_hole circle (at 10 0) (size 2.2 2.2) (drill 1) (layers *.Cu *.Mask)
-      (net 13 "Net-(C5-Pad2)"))
+      (net 14 /NOUT))
     (model ${KISYS3DMOD}/Capacitors_THT.3dshapes/C_Rect_L13.0mm_W5.0mm_P10.00mm_FKS3_FKP3_MKS4.wrl
       (at (xyz 0 0 0))
@@
     )
     (pad 1 thru_hole circle (at 0 0 180) (size 2.2 2.2) (drill 1) (layers *.Cu *.Mask)
-      (net 12 "Net-(C4-Pad1)"))
+      (net 13 /LOUT))
     (pad 2 thru_hole circle (at 10 0 180) (size 2.2 2.2) (drill 1) (layers *.Cu *.Mask)
       (net 6 "Net-(C4-Pad2)"))
@@
     (fp_line (start -19 -13) (end -19 1) (layer F.SilkS) (width 0.15))
     (pad 2 thru_hole oval (at 0 1) (size 6 4) (drill 2) (layers *.Cu *.Mask)
-      (net 12 "Net-(C4-Pad1)"))
+      (net 13 /LOUT))
     (pad 1 thru_hole oval (at -0.02 -13) (size 6 4) (drill 2) (layers *.Cu *.Mask)
       (net 1 /LINE))
@@
     (fp_line (start -19 -13) (end -19 1) (layer F.SilkS) (width 0.15))
     (pad 2 thru_hole oval (at 0 1 180) (size 6 4) (drill 2) (layers *.Cu *.Mask)
-      (net 13 "Net-(C5-Pad2)"))
+      (net 14 /NOUT))
     (pad 1 thru_hole oval (at -0.02 -13 180) (size 6 4) (drill 2) (layers *.Cu *.Mask)
       (net 3 /NEU))
@@
   (segment (start 153 93) (end 153 96) (width 0.8) (layer B.Cu) (net 11))
   (segment (start 153 90) (end 153 93) (width 0.8) (layer B.Cu) (net 11))
-  (segment (start 129.96973 91.00137) (end 129.985323 91.016963) (width 0.8) (layer B.Cu) (net 12))
-  (segment (start 129.985323 91.016963) (end 134.707908 91.016963) (width 0.8) (layer B.Cu) (net 12))
-  (segment (start 134.707908 91.016963) (end 136 92.309055) (width 0.8) (layer B.Cu) (net 12))
-  (segment (start 136 92.309055) (end 136 96.192255) (width 0.8) (layer B.Cu) (net 12))
-  (segment (start 136 96.192255) (end 135.980854 96.211401) (width 0.8) (layer B.Cu) (net 12))
-  (segment (start 129.997788 107.038717) (end 134.78156 107.038717) (width 0.8) (layer B.Cu) (net 13))
-  (segment (start 134.78156 107.038717) (end 136 105.820277) (width 0.8) (layer B.Cu) (net 13))
-  (segment (start 136 105.820277) (end 136 101.737879) (width 0.8) (layer B.Cu) (net 13))
-  (segment (start 136 101.737879) (end 136.007137 101.730742) (width 0.8) (layer B.Cu) (net 13))
-  (segment (start 156 97.5) (end 156 99) (width 0.8) (layer B.Cu) (net 14))
-  (segment (start 156 99) (end 156 100.5) (width 0.8) (layer B.Cu) (net 14))
-  (segment (start 153 99) (end 156 99) (width 0.8) (layer B.Cu) (net 14))
+  (segment (start 156 97.5) (end 156 99) (width 0.8) (layer B.Cu) (net 12))
+  (segment (start 156 99) (end 156 100.5) (width 0.8) (layer B.Cu) (net 12))
+  (segment (start 153 99) (end 156 99) (width 0.8) (layer B.Cu) (net 12))
+  (segment (start 129.96973 91.00137) (end 129.985323 91.016963) (width 0.8) (layer B.Cu) (net 13))
+  (segment (start 129.985323 91.016963) (end 134.707908 91.016963) (width 0.8) (layer B.Cu) (net 13))
+  (segment (start 134.707908 91.016963) (end 136 92.309055) (width 0.8) (layer B.Cu) (net 13))
+  (segment (start 136 92.309055) (end 136 96.192255) (width 0.8) (layer B.Cu) (net 13))
+  (segment (start 136 96.192255) (end 135.980854 96.211401) (width 0.8) (layer B.Cu) (net 13))
+  (segment (start 129.997788 107.038717) (end 134.78156 107.038717) (width 0.8) (layer B.Cu) (net 14))
+  (segment (start 134.78156 107.038717) (end 136 105.820277) (width 0.8) (layer B.Cu) (net 14))
+  (segment (start 136 105.820277) (end 136 101.737879) (width 0.8) (layer B.Cu) (net 14))
+  (segment (start 136 101.737879) (end 136.007137 101.730742) (width 0.8) (layer B.Cu) (net 14))
   (zone (net 2) (net_name Earth) (layer B.Cu) (hatch edge 0.508)
     (connect_pads yes (clearance 0.508))
@@
       )
     )
-  )
-  (zone (net 13) (net_name "Net-(C5-Pad2)") (layer F.Cu) (hatch edge 0.508)
-    (connect_pads yes (clearance 0.508))
-    (min_thickness 0.254)
-    (fill yes (arc_segments 16) (thermal_gap 0.508) (thermal_bridge_width 0.508))
-    (polygon
-      (pts
-        (xy 126 105) (xy 134 105) (xy 134 111) (xy 183 111) (xy 186 108)
-        (xy 186 97) (xy 198 97) (xy 198 100) (xy 188 100) (xy 188 109)
-        (xy 184 113) (xy 126 113)
-      )
-    )
-  )
-  (zone (net 12) (net_name "Net-(C4-Pad1)") (layer F.Cu) (hatch edge 0.508)
-    (connect_pads yes (clearance 0.508))
-    (min_thickness 0.254)
-    (fill yes (arc_segments 16) (thermal_gap 0.508) (thermal_bridge_width 0.508))
-    (polygon
-      (pts
-        (xy 134 89) (xy 118 89) (xy 118 117) (xy 137 117) (xy 137 124)
-        (xy 187 124) (xy 187 116) (xy 192 111) (xy 192 105) (xy 198 105)
-        (xy 198 102) (xy 190 102) (xy 190 110) (xy 185 115) (xy 185 121)
-        (xy 139 121) (xy 139 115) (xy 120 115) (xy 120 91) (xy 125 91)
-        (xy 125 93) (xy 134 93)
-      )
-    )

Commit message: tarpinis kommitas
Other:
- board text added: "LINE"
- board text added: "NEU"
- board text added: "PE"
Changed lines of the file:
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@@
     (area 97.924999 73.924999 199.075001 124.075001)
     (thickness 1.6)
-    (drawings 12)
+    (drawings 18)
     (tracks 54)
     (zones 0)
@@
   (page A4)
   (layers
-    (0 F.Cu signal)
-    (31 B.Cu signal)
+    (0 F.Cu signal hide)
+    (31 B.Cu signal hide)
     (32 B.Adhes user hide)
     (33 F.Adhes user hide)
@@
     (36 B.SilkS user)
     (37 F.SilkS user)
-    (38 B.Mask user)
+    (38 B.Mask user hide)
     (39 F.Mask user hide)
     (40 Dwgs.User user hide)
@@
     )
   )
+  (gr_text PE (at 208.5 93.5) (layer F.SilkS)
+    (effects (font (size 1.5 1.5) (thickness 0.3)))
+  )
+  (gr_text NEU (at 209 103.5) (layer F.SilkS)
+    (effects (font (size 1.5 1.5) (thickness 0.3)))
+  )
+  (gr_text LINE (at 209 98.5) (layer F.SilkS)
+    (effects (font (size 1.5 1.5) (thickness 0.3)))
+  )
+  (gr_text PE (at 88 103.5) (layer F.SilkS)
+    (effects (font (size 1.5 1.5) (thickness 0.3)))
+  )
+  (gr_text NEU (at 88 98.5) (layer F.SilkS)
+    (effects (font (size 1.5 1.5) (thickness 0.3)))
+  )
+  (gr_text LINE (at 88 93.5) (layer F.SilkS)
+    (effects (font (size 1.5 1.5) (thickness 0.3)))
+  )
   (gr_arc (start 199 124) (end 194.5 124) (angle 90) (layer Edge.Cuts) (width 0.15))
